Commit message: added 5 sc poets and sfp,sc_mounts

File: aic_description/urdf/cable.sdf.xacro (robot description, xacro)
@@ -3,4 +3,5 @@
   <xacro:arg name="attach_cable_to_gripper" default="false"/>
   <xacro:arg name="cable_type" default="sfp_sc_cable"/>
+  <xacro:arg name="pin_cable_connection_1" default="false"/>
   <xacro:property name="cable_type" value="$(arg cable_type)" />
   <xacro:property name="end_effector_model" value="ur5e" />
@@ -29,4 +30,5 @@
         <end_effector_link>${end_effector_link}</end_effector_link>
         <create_connection_delay_s>0</create_connection_delay_s>
+        <pin_cable_connection_1>$(arg pin_cable_connection_1)</pin_cable_connection_1>
       </plugin>
       </xacro:if>

File: aic_description/urdf/task_board.urdf.xacro (robot description, xacro)
@@ -51,4 +51,36 @@
   <xacro:arg name="sc_mount_rail_1_pitch" default="0.0"/>
   <xacro:arg name="sc_mount_rail_1_yaw" default="0.0"/>
+  <!-- Additional SFP Mounts: 2/3 on rail 0 side, 4 on rail 1 side -->
+  <xacro:arg name="sfp_mount_rail_2_present" default="false"/>
+  <xacro:arg name="sfp_mount_rail_2_translation" default="0.0"/>
+  <xacro:arg name="sfp_mount_rail_2_roll" default="0.0"/>
+  <xacro:arg name="sfp_mount_rail_2_pitch" default="0.0"/>
+  <xacro:arg name="sfp_mount_rail_2_yaw" default="0.0"/>
+  <xacro:arg name="sfp_mount_rail_3_present" default="false"/>
+  <xacro:arg name="sfp_mount_rail_3_translation" default="0.0"/>
+  <xacro:arg name="sfp_mount_rail_3_roll" default="0.0"/>
+  <xacro:arg name="sfp_mount_rail_3_pitch" default="0.0"/>
+  <xacro:arg name="sfp_mount_rail_3_yaw" default="0.0"/>
+  <xacro:arg name="sfp_mount_rail_4_present" default="false"/>
+  <xacro:arg name="sfp_mount_rail_4_translation" default="0.0"/>
+  <xacro:arg name="sfp_mount_rail_4_roll" default="0.0"/>
+  <xacro:arg name="sfp_mount_rail_4_pitch" default="0.0"/>
+  <xacro:arg name="sfp_mount_rail_4_yaw" default="0.0"/>
+  <!-- Additional SC Mounts: 2/3 on rail 0 side, 4 on rail 1 side -->
+  <xacro:arg name="sc_mount_rail_2_present" default="false"/>
+  <xacro:arg name="sc_mount_rail_2_translation" default="0.0"/>
+  <xacro:arg name="sc_mount_rail_2_roll" default="0.0"/>
+  <xacro:arg name="sc_mount_rail_2_pitch" default="0.0"/>
+  <xacro:arg name="sc_mount_rail_2_yaw" default="0.0"/>
+  <xacro:arg name="sc_mount_rail_3_present" default="false"/>
+  <xacro:arg name="sc_mount_rail_3_translation" default="0.0"/>
+  <xacro:arg name="sc_mount_rail_3_roll" default="0.0"/>
+  <xacro:arg name="sc_mount_rail_3_pitch" default="0.0"/>
+  <xacro:arg name="sc_mount_rail_3_yaw" default="0.0"/>
+  <xacro:arg name="sc_mount_rail_4_present" default="false"/>
+  <xacro:arg name="sc_mount_rail_4_translation" default="0.0"/>
+  <xacro:arg name="sc_mount_rail_4_roll" default="0.0"/>
+  <xacro:arg name="sc_mount_rail_4_pitch" default="0.0"/>
+  <xacro:arg name="sc_mount_rail_4_yaw" default="0.0"/>
   <!-- SC Port 0 -->
   <xacro:arg name="sc_port_0_present" default="false"/>
@@ -63,4 +95,22 @@
   <xacro:arg name="sc_port_1_pitch" default="0.0"/>
   <xacro:arg name="sc_port_1_yaw" default="0.0"/>
+  <!-- SC Port 2 -->
+  <xacro:arg name="sc_port_2_present" default="false"/>
+  <xacro:arg name="sc_port_2_translation" default="0.0"/>
+  <xacro:arg name="sc_port_2_roll" default="0.0"/>
+  <xacro:arg name="sc_port_2_pitch" default="0.0"/>
+  <xacro:arg name="sc_port_2_yaw" default="0.0"/>
+  <!-- SC Port 3 -->
+  <xacro:arg name="sc_port_3_present" default="false"/>
+  <xacro:arg name="sc_port_3_translation" default="0.0"/>
+  <xacro:arg name="sc_port_3_roll" default="0.0"/>
+  <xacro:arg name="sc_port_3_pitch" default="0.0"/>
+  <xacro:arg name="sc_port_3_yaw" default="0.0"/>
+  <!-- SC Port 4 -->
+  <xacro:arg name="sc_port_4_present" default="false"/>
+  <xacro:arg name="sc_port_4_translation" default="0.0"/>
+  <xacro:arg name="sc_port_4_roll" default="0.0"/>
+  <xacro:arg name="sc_port_4_pitch" default="0.0"/>
+  <xacro:arg name="sc_port_4_yaw" default="0.0"/>
   <!-- NIC Card Mount 0 -->
   <xacro:arg name="nic_card_mount_0_present" default="false"/>
@@ -154,4 +204,54 @@
     </joint>
   </xacro:if>
+  <!-- Additional SFP mounts -->
+  <xacro:if value="$(arg sfp_mount_rail_2_present)">
+    <xacro:sfp_mount prefix="sfp_mount_rail_2_"/>
+    <joint name="sfp_mount_rail_2_joint" type="fixed">
+      <parent link="task_board_base_link"/>
+      <child link="sfp_mount_rail_2_link"/>
+      <origin xyz="0.055 ${-0.10625 + $(arg sfp_mount_rail_2_translation)} 0.01" rpy="$(arg sfp_mount_rail_2_roll) $(arg sfp_mount_rail_2_pitch) $(arg sfp_mount_rail_2_yaw)"/>
+    </joint>
+  </xacro:if>
+  <xacro:if value="$(arg sfp_mount_rail_3_present)">
+    <xacro:sfp_mount prefix="sfp_mount_rail_3_"/>
+    <joint name="sfp_mount_rail_3_joint" type="fixed">
+      <parent link="task_board_base_link"/>
+      <child link="sfp_mount_rail_3_link"/>
+      <origin xyz="0.055 ${-0.10625 + $(arg sfp_mount_rail_3_translation)} 0.01" rpy="$(arg sfp_mount_rail_3_roll) $(arg sfp_mount_rail_3_pitch) $(arg sfp_mount_rail_3_yaw)"/>
+    </joint>
+  </xacro:if>
+  <xacro:if value="$(arg sfp_mount_rail_4_present)">
+    <xacro:sfp_mount prefix="sfp_mount_rail_4_"/>
+    <joint name="sfp_mount_rail_4_joint" type="fixed">
+      <parent link="task_board_base_link"/>
+      <child link="sfp_mount_rail_4_link"/>
+      <origin xyz="0.055 ${0.10625 + $(arg sfp_mount_rail_4_translation)} 0.01" rpy="$(arg sfp_mount_rail_4_roll) $(arg sfp_mount_rail_4_pitch) $(arg sfp_mount_rail_4_yaw)"/>
+    </joint>
+  </xacro:if>
+  <!-- Additional SC mounts -->
+  <xacro:if value="$(arg sc_mount_rail_2_present)">
+    <xacro:sc_mount prefix="sc_mount_rail_2_"/>
+    <joint name="sc_mount_rail_2_joint" type="fixed">
+      <parent link="task_board_base_link"/>
+      <child link="sc_mount_rail_2_link"/>
+      <origin xyz="0.1 ${-0.10625 + $(arg sc_mount_rail_2_translation)} 0.012" rpy="$(arg sc_mount_rail_2_roll) $(arg sc_mount_rail_2_pitch) $(arg sc_mount_rail_2_yaw)"/>
+    </joint>
+  </xacro:if>
+  <xacro:if value="$(arg sc_mount_rail_3_present)">
+    <xacro:sc_mount prefix="sc_mount_rail_3_"/>
+    <joint name="sc_mount_rail_3_joint" type="fixed">
+      <parent link="task_board_base_link"/>
+      <child link="sc_mount_rail_3_link"/>
+      <origin xyz="0.1 ${-0.10625 + $(arg sc_mount_rail_3_translation)} 0.012" rpy="$(arg sc_mount_rail_3_roll) $(arg sc_mount_rail_3_pitch) $(arg sc_mount_rail_3_yaw)"/>
+    </joint>
+  </xacro:if>
+  <xacro:if value="$(arg sc_mount_rail_4_present)">
+    <xacro:sc_mount prefix="sc_mount_rail_4_"/>
+    <joint name="sc_mount_rail_4_joint" type="fixed">
+      <parent link="task_board_base_link"/>
+      <child link="sc_mount_rail_4_link"/>
+      <origin xyz="0.0985 ${0.10625 + $(arg sc_mount_rail_4_translation)} 0.01" rpy="$(arg sc_mount_rail_4_roll) $(arg sc_mount_rail_4_pitch) $(arg sc_mount_rail_4_yaw)"/>
+    </joint>
+  </xacro:if>
   <!-- SC Port 0 -->
   <xacro:if value="$(arg sc_port_0_present)">
@@ -164,11 +264,41 @@
     </gazebo>
   </xacro:if>
-  <!-- SC Port 1 -->
+  <!-- SC Port 1 (SC rail 0) -->
   <xacro:if value="$(arg sc_port_1_present)">
-    <xacro:sc_port prefix="sc_port_1" pose="${-0.075 + $(arg sc_port_1_translation)} 0.0705 0.0165 ${1.57 + $(arg sc_port_1_roll)} $(arg sc_port_1_pitch) ${1.57 + $(arg sc_port_1_yaw)}"/>
+    <xacro:sc_port prefix="sc_port_1" pose="${-0.075 + $(arg sc_port_1_translation)} 0.0295 0.0165 ${1.57 + $(arg sc_port_1_roll)} $(arg sc_port_1_pitch) ${1.57 + $(arg sc_port_1_yaw)}"/>
     <gazebo>
       <joint name="sc_port_1_joint" type="fixed">
         <parent>task_board_base_link</parent>
         <child>sc_port_1::sc_port_link</child>
+      </joint>
+    </gazebo>
+  </xacro:if>
+  <!-- SC Port 2 (SC rail 0) -->
+  <xacro:if value="$(arg sc_port_2_present)">
+    <xacro:sc_port prefix="sc_port_2" pose="${-0.075 + $(arg sc_port_2_translation)} 0.0295 0.0165 ${1.57 + $(arg sc_port_2_roll)} $(arg sc_port_2_pitch) ${1.57 + $(arg sc_port_2_yaw)}"/>
+    <gazebo>
+      <joint name="sc_port_2_joint" type="fixed">
+        <parent>task_board_base_link</parent>
+        <child>sc_port_2::sc_port_link</child>
+      </joint>
+    </gazebo>
+  </xacro:if>
+  <!-- SC Port 3 (SC rail 1) -->
+  <xacro:if value="$(arg sc_port_3_present)">
+    <xacro:sc_port prefix="sc_port_3" pose="${-0.075 + $(arg sc_port_3_translation)} 0.0705 0.0165 ${1.57 + $(arg sc_port_3_roll)} $(arg sc_port_3_pitch) ${1.57 + $(arg sc_port_3_yaw)}"/>
+    <gazebo>
+      <joint name="sc_port_3_joint" type="fixed">
+        <parent>task_board_base_link</parent>
+        <child>sc_port_3::sc_port_link</child>
+      </joint>
+    </gazebo>
+  </xacro:if>
+  <!-- SC Port 4 (SC rail 1) -->
+  <xacro:if value="$(arg sc_port_4_present)">
+    <xacro:sc_port prefix="sc_port_4" pose="${-0.075 + $(arg sc_port_4_translation)} 0.0705 0.0165 ${1.57 + $(arg sc_port_4_roll)} $(arg sc_port_4_pitch) ${1.57 + $(arg sc_port_4_yaw)}"/>
+    <gazebo>
+      <joint name="sc_port_4_joint" type="fixed">
+        <parent>task_board_base_link</parent>
+        <child>sc_port_4::sc_port_link</child>
       </joint>
     </gazebo>
